File: schematics/LedMatrixSensorNode/LedMatrixSensorNode.kicad_sch (KiCad schematic)
At the start: 13 parts, among them J1 LED2, J2 BH1750, J3 SCD41, J4 HTU21D, J5 HLK-LD2450, J6 HLK-LD2410, J7 Beeper, J8 Power + Buttons, J9 LED, U2 DC/DC, U8 XIAO-ESP32-S3-Plus-SMD

Commit message: Updated schematics
Parts:
- added U7: DC/DC 3.3v, symbol Regulator_Linear:L7805
- J6: value HLK-LD2410 -> HLK-LD2412
- U2: value DC/DC -> DC/DC 3.3v
Connections:
- net at J2.1 (Pin_1), J3.2 (Pin_2), J4.1 (Pin_1)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: no longer J6.1 (Pin_1), J8.1 (Pin_1)
- net at J2.2 (Pin_2), J5.4 (Pin_4), J6.3 (Pin_3)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: now also U7.2 (GND)
- net at U2.1 (IN), U8.14 (VBUS): now also J6.1 (Pin_1), U7.1 (IN)
- new net: J8.1 (Pin_1), U7.3 (OUT)
Other:
- moved on the sheet: R1, R2

Commit message: WIP HLK-LD2454 room presence
Parts:
- J5: value HLK-LD2450 -> HLK-LD2454
Connections:
- net at J2.1 (Pin_1), J3.2 (Pin_2), J4.1 (Pin_1)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: no longer J5.1 (Pin_1)
- net RADAR_R: now reaches J5.2 (Pin_2), U8.8 (GPIO44_D7_RX)
- net RADAR_T: now reaches J5.3 (Pin_3), U8.21 (GPIO11_DVP_Y8_SPI_MOSI1)
- net at J2.2 (Pin_2), J5.4 (Pin_4), J6.3 (Pin_3)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: now also J3.1 (Pin_1), J4.2 (Pin_2), J7.2 (Pin_2), U8.13 (GND)
- net at J6.1 (Pin_1), U2.1 (IN), U7.1 (IN)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: now also J5.1 (Pin_1)
Other:
- note added: "Radar header (HLK-LD2454) to radar J1 [1 5V, 2 G, 3 T, 4 R] - the cable is NOT 1:1: header 1 VBUS -> J1-1 5V (LD2454 manual: DC 5 V, >200 mA) header 4 GND -> J1-2 G header 3 RADAR_T -> J1-3 T (radar TX -> GPIO11 / Serial1 RX) header 2 RADAR_R -> J1-4 R (radar RX <- D7 / GPIO44 / Serial1 TX, needed to enable multi-target mode)"
Changed lines of the file:
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@@
 	(generator_version "10.0")
 	(paper "A4")
+	(text "Radar header (HLK-LD2454) to radar J1 [1 5V, 2 G, 3 T, 4 R] - the cable is NOT 1:1:\n  header 1  VBUS     -> J1-1 5V  (LD2454 manual: DC 5 V, >200 mA)\n  header 4  GND      -> J1-2 G\n  header 3  RADAR_T  -> J1-3 T  (radar TX -> GPIO11 / Serial1 RX)\n  header 2  RADAR_R  -> J1-4 R  (radar RX <- D7 / GPIO44 / Serial1 TX, needed to enable multi-target mode)"
+		(exclude_from_sim no)
+		(at 127 132.08 0)
+		(effects
+			(font
+				(size 1.27 1.27)
+			)
+			(justify left top)
+		)
+	)
 	(junction
 		(at 218.44 81.28)
@@
 	)
 	(junction
+		(at 199.39 49.53)
+		(diameter 0)
+		(color 0 0 0 0)
+	)
+	(junction
 		(at 196.85 86.36)
 		(diameter 0)
@@
 	)
 	(junction
+		(at 226.06 86.36)
+		(diameter 0)
+		(color 0 0 0 0)
+	)
+	(junction
 		(at 213.36 121.92)
 		(diameter 0)
@@
 	(wire
 		(pts
-			(xy 231.14 67.31) (xy 231.14 73.66)
-		)
-		(stroke
-			(width 0)
-			(type default)
-		)
-	)
-	(wire
-		(pts
 			(xy 212.09 52.07) (xy 212.09 59.69)
 		)
@@
 	(wire
 		(pts
-			(xy 196.85 86.36) (xy 236.22 86.36)
+			(xy 196.85 86.36) (xy 226.06 86.36)
 		)
 		(stroke
@@
 	(wire
 		(pts
+			(xy 226.06 73.66) (xy 226.06 86.36)
+		)
+		(stroke
+			(width 0)
+			(type default)
+		)
+	)
+	(wire
+		(pts
 			(xy 38.1 58.42) (xy 38.1 57.15)
 		)
@@
 	(wire
 		(pts
-			(xy 231.14 73.66) (xy 236.22 73.66)
-		)
-		(stroke
-			(width 0)
-			(type default)
-		)
-	)
-	(wire
-		(pts
 			(xy 209.55 54.61) (xy 209.55 62.23)
 		)
@@
 	(wire
 		(pts
+			(xy 199.39 49.53) (xy 199.39 33.02)
+		)
+		(stroke
+			(width 0)
+			(type default)
+		)
+	)
+	(wire
+		(pts
 			(xy 223.52 105.41) (xy 223.52 106.68)
 		)
@@
 	(wire
 		(pts
+			(xy 226.06 73.66) (xy 236.22 73.66)
+		)
+		(stroke
+			(width 0)
+			(type default)
+		)
+	)
+	(wire
+		(pts
 			(xy 238.76 109.22) (xy 238.76 124.46)
 		)
@@
 	(wire
 		(pts
+			(xy 226.06 86.36) (xy 236.22 86.36)
+		)
+		(stroke
+			(width 0)
+			(type default)
+		)
+	)
+	(wire
+		(pts
 			(xy 254 55.88) (xy 254 59.69)
 		)
@@
 			(width 0)
 			(type default)
+		)
+	)
+	(label "RADAR_T"
+		(at 236.22 78.74 180)
+		(effects
+			(font
+				(size 1.27 1.27)
+			)
+			(justify right bottom)
+		)
+	)
+	(label "RADAR_R"
+		(at 236.22 76.2 180)
+		(effects
+			(font
+				(size 1.27 1.27)
+			)
+			(justify right bottom)
 		)
 	)
@@
 			)
 		)
-		(property "Value" "HLK-LD2450"
+		(property "Value" "HLK-LD2454"
 			(at 243.84 77.4699 0)
 			(show_name no)
